File: monitor.brd (EAGLE design)
At the start: 148.1 x 84.8 mm, 72 parts, among them IC1 LM1117-5, IC2 LM1117-5, J3 DCJ0202, J4 DCJ0202, J5 DCJ0202, Q1 IRLML2502, T1 BC846, T2 BT148, X3 PN61729-S, X4 PN87520-S

Commit message: drill sizes
Parts:
- moved SJ2 0.51 mm to (77.7, 76.2)
- moved C6 0.25 mm to (77.7, 79.8)
- moved JP3 0.25 mm to (77.5, 73.4)
Routing:
- net +5V: track 141.4 -> 142.0 mm
Changed lines of the file:
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@@
 <setting verticaltext="up"/>
 </settings>
-<grid distance="10" unitdist="mil" unit="mil" style="lines" multiple="1" display="yes" altdistance="200" altunitdist="mil" altunit="mil"/>
+<grid distance="10" unitdist="mil" unit="mil" style="lines" multiple="1" display="yes" altdistance="1" altunitdist="mil" altunit="mm"/>
 <layers>
 <layer number="1" name="Top" color="4" fill="1" visible="yes" active="yes"/>
@@
 </element>
 <element name="C5" library="rcl" package="SMC_B" value="100u" x="67.31" y="78.994" rot="R270"/>
-<element name="C6" library="rcl" package="SMC_B" value="100u" x="77.724" y="79.502" rot="R90"/>
+<element name="C6" library="rcl" package="SMC_B" value="100u" x="77.724" y="79.756" rot="R90"/>
 <element name="IC1" library="burr-brown" package="SOT223" value="LM1117-5" x="72.39" y="77.724" rot="R180">
 <attribute name="OC_NEWARK" value="14P6981" x="53.34" y="275.844" size="1.778" layer="27" rot="R180" display="off"/>
@@
 </element>
 <element name="JP2" library="jumper" package="JP2" value="" x="47.244" y="73.66"/>
-<element name="JP3" library="jumper" package="JP1" value="" x="77.47" y="73.152" rot="R90"/>
+<element name="JP3" library="jumper" package="JP1" value="" x="77.47" y="73.406" rot="R90"/>
 <element name="IC2" library="burr-brown" package="SOT223" value="LM1117-5" x="39.878" y="78.74">
 <attribute name="OC_NEWARK" value="14P6981" x="67.818" y="-119.38" size="1.778" layer="27" display="off"/>
@@
 <element name="C8" library="rcl" package="SMC_B" value="100u" x="46.736" y="78.74" rot="R90"/>
 <element name="C9" library="rcl" package="SMC_B" value="100u" x="34.798" y="78.74" rot="R270"/>
-<element name="SJ2" library="jumper" package="SJ" value="" x="77.724" y="75.692" rot="R180"/>
+<element name="SJ2" library="jumper" package="SJ" value="" x="77.724" y="76.2" rot="R180"/>
 <element name="C11" library="rcl" package="C0603" value="100n" x="58.674" y="65.786"/>
 <element name="C12" library="rcl" package="C0603" value="100n" x="58.166" y="60.706" rot="R90"/>
@@
 <wire x1="56.16" y1="74.93" x2="56.16" y2="77.19" width="0.6096" layer="16"/>
 <wire x1="48.768" y1="82.296" x2="46.736" y2="82.296" width="0.6096" layer="16"/>
-<wire x1="80.542" y1="81.002" x2="83.058" y2="78.486" width="0.6096" layer="1"/>
 <wire x1="139.512" y1="68.26" x2="140.904" y2="68.26" width="0.6096" layer="1"/>
 <wire x1="140.904" y1="68.26" x2="140.97" y2="68.326" width="0.6096" layer="1"/>
 <via x="140.97" y="68.326" extent="1-16" drill="0.6"/>
-<wire x1="77.724" y1="81.002" x2="77.5956" y2="80.8736" width="0.6096" layer="1"/>
 <wire x1="77.5956" y1="80.8736" x2="74.6506" y2="80.8736" width="0.6096" layer="1"/>
-<wire x1="80.542" y1="81.002" x2="77.724" y2="81.002" width="0.6096" layer="1"/>
 <wire x1="32.766" y1="74.422" x2="34.29" y2="74.422" width="0.8128" layer="16"/>
 <wire x1="46.736" y1="82.296" x2="33.02" y2="82.296" width="0.8128" layer="16"/>
@@
 <wire x1="22.7076" y1="32.0548" x2="17.6276" y2="32.0548" width="0.4064" layer="16"/>
 <wire x1="17.6276" y1="32.0548" x2="10.16" y2="39.5224" width="0.4064" layer="16"/>
+<wire x1="83.058" y1="78.486" x2="80.288" y2="81.256" width="0.6096" layer="1"/>
+<wire x1="80.288" y1="81.256" x2="77.724" y2="81.256" width="0.6096" layer="1"/>
 </signal>
 <signal name="SPI2_NSS">
@@
 <wire x1="102.362" y1="62.992" x2="126.848" y2="62.992" width="0.6096" layer="1"/>
 <wire x1="126.848" y1="62.992" x2="128.372" y2="64.516" width="0.6096" layer="1"/>
-<wire x1="76.962" y1="75.692" x2="76.962" y2="73.914" width="0.6096" layer="1"/>
-<wire x1="76.962" y1="73.914" x2="76.2" y2="73.152" width="0.6096" layer="1"/>
+<wire x1="76.962" y1="76.2" x2="76.962" y2="74.168" width="0.6096" layer="1"/>
 <wire x1="69.342" y1="68.326" x2="60.198" y2="68.326" width="0.6096" layer="1"/>
 <wire x1="60.198" y1="68.326" x2="58.166" y2="70.358" width="0.6096" layer="1"/>
-<wire x1="76.2" y1="73.152" x2="75.438" y2="73.152" width="0.6096" layer="1"/>
-<wire x1="75.438" y1="73.152" x2="74.422" y2="72.136" width="0.6096" layer="1"/>
+<wire x1="75.692" y1="73.406" x2="74.422" y2="72.136" width="0.6096" layer="1"/>
 <wire x1="74.422" y1="72.136" x2="73.152" y2="72.136" width="0.6096" layer="1"/>
 <wire x1="73.152" y1="72.136" x2="69.342" y2="68.326" width="0.6096" layer="1"/>
@@
 <wire x1="85.598" y1="25.146" x2="85.598" y2="27.686" width="0.6096" layer="1"/>
 <wire x1="83.82" y1="64.262" x2="85.598" y2="62.484" width="0.8128" layer="1"/>
-<wire x1="76.2" y1="73.152" x2="76.2" y2="71.882" width="0.6096" layer="16"/>
+<wire x1="76.2" y1="73.406" x2="76.2" y2="71.882" width="0.6096" layer="16"/>
 <wire x1="76.2" y1="71.882" x2="83.82" y2="64.262" width="0.6096" layer="16"/>
 <wire x1="51.562" y1="73.66" x2="49.784" y2="73.66" width="0.6096" layer="1"/>
+<wire x1="75.692" y1="73.406" x2="76.2" y2="73.406" width="0.6096" layer="1"/>
+<wire x1="76.2" y1="73.406" x2="76.962" y2="74.168" width="0.6096" layer="1"/>
 </signal>
 <signal name="!RST">
@@
 <wire x1="72.81" y1="82.804" x2="72.81" y2="81.319" width="0.6096" layer="1"/>
 <wire x1="72.81" y1="81.319" x2="72.3646" y2="80.8736" width="0.6096" layer="1"/>
-<wire x1="77.724" y1="78.002" x2="78.486" y2="77.24" width="0.6096" layer="1"/>
-<wire x1="78.486" y1="77.24" x2="78.486" y2="75.692" width="0.6096" layer="1"/>
-<wire x1="77.724" y1="78.002" x2="73.89" y2="78.002" width="0.6096" layer="1"/>
-<wire x1="73.89" y1="78.002" x2="72.39" y2="79.502" width="0.6096" layer="1"/>
+<wire x1="78.486" y1="77.24" x2="78.486" y2="76.2" width="0.6096" layer="1"/>
 <wire x1="72.39" y1="79.502" x2="72.39" y2="80.8482" width="0.6096" layer="1"/>
 <wire x1="72.39" y1="80.8482" x2="72.3646" y2="80.8736" width="0.6096" layer="1"/>
-<wire x1="78.486" y1="75.692" x2="78.486" y2="73.406" width="0.6096" layer="1"/>
-<wire x1="78.486" y1="73.406" x2="78.74" y2="73.152" width="0.6096" layer="1"/>
+<wire x1="78.486" y1="76.2" x2="78.486" y2="73.406" width="0.6096" layer="1"/>
+<wire x1="78.486" y1="73.406" x2="78.74" y2="73.406" width="0.6096" layer="1"/>
+<wire x1="72.39" y1="79.502" x2="73.636" y2="78.256" width="0.6096" layer="1"/>
+<wire x1="73.636" y1="78.256" x2="77.724" y2="78.256" width="0.6096" layer="1"/>
+<wire x1="78.486" y1="77.24" x2="77.724" y2="78.002" width="0.6096" layer="1"/>
+<wire x1="77.724" y1="78.002" x2="77.724" y2="78.256" width="0.6096" layer="1"/>
 </signal>
 <signal name="V_SUPPLY">
