File: monitor.sch (EAGLE design)
At the start: 72 parts, among them IC1 LM1117-5, IC2 LM1117-5, J3 DCJ0202, J4 DCJ0202, J5 DCJ0202, Q1 IRLML2502, T1 BC846, T2 BT148, X3 PN61729-S, X4 PN87520-S

Commit message: condensators, minor layout changes
Parts:
- added C17: 10u, rcl:C-EUC1206
- added C18, C19: 100n, rcl:C-EUC0603
- F1: value 500m -> 1A
Connections:
- net +5V: now also C17.1
- net B_ESC: now also U$1G$2.PD6; no longer U$1G$2.PB5
- net GND: now also C17.2, C18.2, C19.2
- net N$13: now also C19.1
- net OUT: now also C18.1
Other:
- moved on the sheet: D1, D3
